File: aardvark-i2c-breakout.kicad_sch (KiCad schematic)
At the start: 2 parts, among them J1 Conn_02x05_Odd_Even, J2 Conn_01x03

Commit message: Title block
Other:
- title: (none) -> Aardvark I2C Breakout
Changed lines of the file:
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@@
 (kicad_sch (version 20230121) (generator eeschema)
-  (paper "A4")
+  (paper "USLetter")
+  (title_block
+    (title "Aardvark I2C Breakout")
+    (date "2023-02-18")
+    (rev "1.0")
+  )
   (no_connect (at 148.59 93.98))
   (no_connect (at 148.59 96.52))
@@
     (pin "3")
     (instances
-      (project "AardvarkBreakout"
+      (project "aardvark-i2c-breakout"
         (path "/dd35b9f1-2797-46a7-a3ff-4e2c1be5fc91"
           (reference "J2") (unit 1)
@@
     (pin "9")
     (instances
-      (project "AardvarkBreakout"
+      (project "aardvark-i2c-breakout"
         (path "/dd35b9f1-2797-46a7-a3ff-4e2c1be5fc91"
           (reference "J1") (unit 1)
